File: src/fanController.brd (EAGLE design)
At the start: 41.9 x 38.1 mm, 20 parts, among them IC1 MIC4420M, Q1 MOSFET-NCHANNELFDD8780

Commit message: Updated Rev B for production.
Parts:
- added C1, C2: 0.1uF, resistor:C0805
- IC2: value (none) -> NE555
- R5: value TSR-3386 -> TSR-3386-100K
- moved IC1 2.54 mm to (31.8, 26.7)
- moved R4 2.54 mm to (23.2, 28.3)
- moved C5 1.92 mm to (21.9, 12.0)
- flipped U$2 to the bottom
Connections:
- net GND: now also C1.2, C2.2
- net VCC: now also C1.1, C2.1
Routing:
- net VCC: track 45.5 -> 55.7 mm, vias 2 -> 0
- net N$3: track 10.9 -> 8.32 mm
- net CNTRL: track 33.2 -> 35.5 mm
Other:
- board text added: "B"
- board text added: "DC PWM Controler"
- board text removed: "A"
- board text removed: "Fan Controler"
