File: src/fanController.brd (EAGLE design)
At the start: 41.9 x 38.1 mm, 22 parts, among them IC1 MIC4420M, IC2 NE555, Q1 MOSFET-NCHANNELFDD8780

Commit message: Update 10nF cap to 1nF
Parts:
- C5: value 10nF -> 1nF
Changed lines of the file:
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@@
 <attribute name="VALUE" x="19.7625" y="4.615" size="1.27" layer="27" rot="R90"/>
 </element>
-<element name="C5" library="resistor" package="C0805" value="10nF" x="21.9075" y="12.0015" smashed="yes" rot="R90">
+<element name="C5" library="resistor" package="C0805" value="1nF" x="21.9075" y="12.0015" smashed="yes" rot="R90">
 <attribute name="NAME" x="19.558" y="11.4935" size="0.8128" layer="25"/>
 <attribute name="VALUE" x="24.1935" y="11.1125" size="1.27" layer="27" rot="R90"/>
