File: src/fanController.sch (EAGLE design)
At the start: 20 parts, among them IC1 MIC4420M, IC2 NE555, Q1 MOSFET-NCHANNELFDD8780

Commit message: Minos adjustments to schematic.
Parts:
- C5: value 10nF -> 1nF
Changed lines of the file:
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@@
 <part name="D4" library="diode" deviceset="MBR0520LT" device=""/>
 <part name="D5" library="diode" deviceset="MBR0520LT" device=""/>
-<part name="C5" library="resistor" deviceset="C-EU" device="C0805" value="10nF"/>
+<part name="C5" library="resistor" deviceset="C-EU" device="C0805" value="1nF"/>
 <part name="C6" library="resistor" deviceset="C-EU" device="C0805" value="10nF"/>
 <part name="C7" library="resistor" deviceset="C-EU" device="C0805" value="0.1uF"/>
