File: src/fanController.sch (EAGLE design)
At the start: 18 parts, among them Q1 MOSFET-NCHANNELFDD8780

Commit message: Updated final version.
Parts:
- removed R2: 47K, pot:TRIM_EU-B64Y
- added R3: TSR-3386, SparkFun-Electromechanical:TRIMPOT-PTH-KNOB
Connections:
- net N$2: now also R3.CW; no longer R2.A
- net N$4: now also R3.WIPER; no longer R2.S
- net N$6: now also R3.CCW; no longer R2.E
Changed lines of the file:
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@@
 <layers>
 <layer number="1" name="Top" color="4" fill="1" visible="no" active="no"/>
+<layer number="2" name="Route2" color="1" fill="3" visible="no" active="no"/>
+<layer number="3" name="Route3" color="4" fill="3" visible="no" active="no"/>
+<layer number="14" name="Route14" color="1" fill="6" visible="no" active="no"/>
+<layer number="15" name="Route15" color="4" fill="6" visible="no" active="no"/>
 <layer number="16" name="Bottom" color="1" fill="1" visible="no" active="no"/>
 <layer number="17" name="Pads" color="2" fill="1" visible="no" active="no"/>
@@
 <part name="STANDOFF3" library="SparkFun-Electromechanical" deviceset="STAND-OFF" device="TIGHT" value="STAND-OFFTIGHT"/>
 <part name="STANDOFF4" library="SparkFun-Electromechanical" deviceset="STAND-OFF" device="TIGHT" value="STAND-OFFTIGHT"/>
-<part name="R2" library="pot" deviceset="TRIM_EU-" device="B64Y" value="47K"/>
+<part name="R3" library="SparkFun-Electromechanical" deviceset="TRIMPOT" device="-PTH-KNOB" value="TSR-3386"/>
 </parts>
 <sheets>
 <sheet>
 <plain>
-<text x="25.4" y="63.5" size="1.778" layer="97">PTD901-1015F-B203</text>
+<text x="30.734" y="62.484" size="1.778" layer="97">PTD901-1015F-B203</text>
 </plain>
 <instances>
@@
 <instance part="STANDOFF3" gate="G$1" x="58.42" y="17.78"/>
 <instance part="STANDOFF4" gate="G$1" x="63.5" y="17.78"/>
-<instance part="R2" gate="1" x="43.18" y="73.66" smashed="yes" rot="R270">
-<attribute name="NAME" x="46.99" y="69.469" size="1.778" layer="95"/>
-<attribute name="VALUE" x="39.37" y="77.47" size="1.778" layer="96"/>
+<instance part="R3" gate="R?" x="43.18" y="73.66" smashed="yes" rot="R180">
+<attribute name="NAME" x="54.61" y="72.1614" size="1.778" layer="95" rot="R180"/>
+<attribute name="VALUE" x="49.022" y="67.818" size="1.778" layer="96" rot="R180"/>
 </instance>
 </instances>
@@
 <wire x1="78.74" y1="68.58" x2="68.58" y2="68.58" width="0.1524" layer="91"/>
 <junction x="68.58" y="68.58"/>
-<pinref part="R2" gate="1" pin="S"/>
 <wire x1="43.18" y1="68.58" x2="68.58" y2="68.58" width="0.1524" layer="91"/>
+<pinref part="R3" gate="R?" pin="WIPER"/>
 </segment>
 </net>
@@
 <segment>
 <pinref part="D1" gate="G$1" pin="A"/>
-<pinref part="R2" gate="1" pin="A"/>
 <wire x1="38.1" y1="78.74" x2="38.1" y2="73.66" width="0.1524" layer="91"/>
+<pinref part="R3" gate="R?" pin="CW"/>
 </segment>
 </net>
@@
 <segment>
 <pinref part="D2" gate="G$1" pin="C"/>
-<pinref part="R2" gate="1" pin="E"/>
 <wire x1="48.26" y1="78.74" x2="48.26" y2="73.66" width="0.1524" layer="91"/>
-</segment>
-</net>
+<pinref part="R3" gate="R?" pin="CCW"/>
+</segment>
+</net>

Commit message: Updated documentation and layout.
Parts:
- Q1: value MOSFET-NCHANNELFDD8780 -> IPD90N03S4L-03
- R1: value 4K7 -> 1K
Other:
- note added: "A"
- note added: "DC Dimmer controller"
- note added: "License: CERN OSHWReleased under the CERN Open Hardware Licence v1.2 http://www.ohwr.org/attachments/2388/cern_ohl_v_1_2.txt Copyright (c) 2017 - by F. Malpartida"
- note added: "PTD901-2015K-B104 - 100K"
- note removed: "PTD901-1015F-B203"
Changed lines of the file:
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@@
 <?xml version="1.0" encoding="utf-8"?>
 <!DOCTYPE eagle SYSTEM "eagle.dtd">
-<eagle version="7.6.0">
+<eagle version="8.1.0">
 <drawing>
 <settings>
@@
 <part name="IC1" library="SparkFun-AnalogIC" deviceset="NE555" device="D"/>
 <part name="FRAME1" library="frames" deviceset="DINA4_L" device=""/>
-<part name="R1" library="resistor" deviceset="R-EU_" device="M0805" value="4K7"/>
+<part name="R1" library="resistor" deviceset="R-EU_" device="M0805" value="1K"/>
 <part name="GND1" library="supply1" deviceset="GND" device=""/>
 <part name="P+1" library="supply1" deviceset="VCC" device=""/>
@@
 <part name="D3" library="diode" deviceset="MBR0520LT" device=""/>
 <part name="P+4" library="supply1" deviceset="VCC" device=""/>
-<part name="Q1" library="SparkFun-DiscreteSemi" deviceset="MOSFET-NCHANNEL" device="FDD8780"/>
+<part name="Q1" library="SparkFun-DiscreteSemi" deviceset="MOSFET-NCHANNEL" device="FDD8780" value="IPD90N03S4L-03"/>
 <part name="GND4" library="supply1" deviceset="GND" device=""/>
 <part name="R4" library="resistor" deviceset="R-EU_" device="M0805" value="22R"/>
@@
 <sheet>
 <plain>
-<text x="30.734" y="62.484" size="1.778" layer="97">PTD901-1015F-B203</text>
+<text x="21.844" y="62.992" size="1.778" layer="97">PTD901-2015K-B104 - 100K</text>
+<text x="83.82" y="154.94" size="5.08" layer="97" ratio="12">DC Dimmer controller</text>
+<text x="256.54" y="7.62" size="2.54" layer="97" ratio="12">A</text>
+<text x="45.72" y="22.86" size="1.778" layer="97" ratio="12">License: CERN OSHWReleased under the CERN Open Hardware Licence v1.2
+http://www.ohwr.org/attachments/2388/cern_ohl_v_1_2.txt
+Copyright (c) 2017 - by F. Malpartida </text>
 </plain>
 <instances>
@@
 <instance part="GND2" gate="1" x="68.58" y="53.34"/>
 <instance part="D1" gate="G$1" x="38.1" y="81.28" smashed="yes" rot="R90">
-<attribute name="NAME" x="36.0934" y="80.264" size="1.778" layer="95" rot="R90"/>
-<attribute name="VALUE" x="33.8074" y="68.58" size="1.778" layer="96" rot="R90"/>
+<attribute name="NAME" x="39.37" y="88.1634" size="1.778" layer="95" rot="R180"/>
+<attribute name="VALUE" x="34.8234" y="73.152" size="1.778" layer="96" rot="R90"/>
 </instance>
 <instance part="D2" gate="G$1" x="48.26" y="81.28" smashed="yes" rot="R270">
-<attribute name="NAME" x="50.0126" y="85.852" size="1.778" layer="95" rot="R270"/>
-<attribute name="VALUE" x="52.8066" y="85.852" size="1.778" layer="96" rot="R270"/>
+<attribute name="NAME" x="46.482" y="85.5726" size="1.778" layer="95"/>
+<attribute name="VALUE" x="50.2666" y="88.392" size="1.778" layer="96" rot="R270"/>
 </instance>
 <instance part="X1" gate="-1" x="96.52" y="124.46"/>
@@
 </schematic>
 </drawing>
+<compatibility>
+<note version="6.3" minversion="6.2.2" severity="warning">
+Since Version 6.2.2 text objects can contain more than one line,
+which will not be processed correctly with this version.
+</note>
+</compatibility>
 </eagle>

Commit message: Schematic touchups for final release after testing. Added alternative values to the schematics.
Parts:
- C3: value 10nF -> 1nF
- R1: value 1K -> 100R
Other:
- note added: "220uF for higher current switching."
- note added: "Between 22R and 100R"
Changed lines of the file:
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@@
 <?xml version="1.0" encoding="utf-8"?>
 <!DOCTYPE eagle SYSTEM "eagle.dtd">
-<eagle version="8.1.0">
+<eagle version="7.6.0">
 <drawing>
 <settings>
@@
 <part name="IC1" library="SparkFun-AnalogIC" deviceset="NE555" device="D"/>
 <part name="FRAME1" library="frames" deviceset="DINA4_L" device=""/>
-<part name="R1" library="resistor" deviceset="R-EU_" device="M0805" value="1K"/>
+<part name="R1" library="resistor" deviceset="R-EU_" device="M0805" value="100R"/>
 <part name="GND1" library="supply1" deviceset="GND" device=""/>
 <part name="P+1" library="supply1" deviceset="VCC" device=""/>
 <part name="C1" library="resistor" deviceset="C-EU" device="C0805" value="0.1uF"/>
 <part name="C2" library="resistor" deviceset="C-EU" device="C0805" value="10nF"/>
-<part name="C3" library="resistor" deviceset="C-EU" device="C0805" value="10nF"/>
+<part name="C3" library="resistor" deviceset="C-EU" device="C0805" value="1nF"/>
 <part name="P+2" library="supply1" deviceset="VCC" device=""/>
 <part name="GND2" library="supply1" deviceset="GND" device=""/>
@@
 http://www.ohwr.org/attachments/2388/cern_ohl_v_1_2.txt
 Copyright (c) 2017 - by F. Malpartida </text>
+<text x="116.84" y="116.84" size="1.9304" layer="97" ratio="12">220uF for higher current switching.</text>
+<text x="137.16" y="60.96" size="1.9304" layer="97" ratio="12">Between 22R and 100R</text>
 </plain>
 <instances>
